Commit message: added dreamwaq

File: src/robots/go2_description/urdf/go2_description.urdf (robot description, URDF)
Before this commit: robot go2_description, 30 links, 29 joints
Joints:
- joint FL_calf_joint: limit lower=-2.7227 upper=-0.83776 effort=45.43 velocity=15.70 -> lower=-2.7227 upper=-0.83776 effort=23.7 velocity=15.70
- joint FR_calf_joint: limit lower=-2.7227 upper=-0.83776 effort=45.43 velocity=15.70 -> lower=-2.7227 upper=-0.83776 effort=23.7 velocity=15.70
- joint RL_calf_joint: limit lower=-2.7227 upper=-0.83776 effort=45.43 velocity=15.70 -> lower=-2.7227 upper=-0.83776 effort=23.7 velocity=15.70
- joint RR_calf_joint: limit lower=-2.7227 upper=-0.83776 effort=45.43 velocity=15.70 -> lower=-2.7227 upper=-0.83776 effort=23.7 velocity=15.70

File: src/robots/go2_description/xacro/gazebo.xacro (robot description, xacro)
@@ -3,5 +3,6 @@
     <xacro:property name="hip_torque_max" value="23.7"/>
     <xacro:property name="thigh_torque_max" value="23.7"/>
-    <xacro:property name="calf_torque_max" value="35.55"/>
+    <!-- <xacro:property name="calf_torque_max" value="35.55"/> -->
+    <xacro:property name="calf_torque_max" value="23.7"/>
     <xacro:property name="ros_version" value="$(env ROS_VERSION)" />
     <xacro:if value="${int(ros_version) == 1}">

Commit message: fix jumping when transition from stand to walk

File: src/robots/go2_description/urdf/go2_description.urdf (robot description, URDF)
Before this commit: robot go2_description, 30 links, 29 joints
Joints:
- joint FL_calf_joint: limit lower=-2.7227 upper=-0.83776 effort=23.7 velocity=15.70 -> lower=-2.7227 upper=-0.83776 effort=45.43 velocity=30.1
- joint FR_calf_joint: limit lower=-2.7227 upper=-0.83776 effort=23.7 velocity=15.70 -> lower=-2.7227 upper=-0.83776 effort=45.43 velocity=30.1
- joint RL_calf_joint: limit lower=-2.7227 upper=-0.83776 effort=23.7 velocity=15.70 -> lower=-2.7227 upper=-0.83776 effort=45.43 velocity=30.1
- joint RR_calf_joint: limit lower=-2.7227 upper=-0.83776 effort=23.7 velocity=15.70 -> lower=-2.7227 upper=-0.83776 effort=45.43 velocity=30.1

File: src/robots/go2_description/xacro/gazebo.xacro (robot description, xacro)
@@ -3,6 +3,6 @@
     <xacro:property name="hip_torque_max" value="23.7"/>
     <xacro:property name="thigh_torque_max" value="23.7"/>
-    <!-- <xacro:property name="calf_torque_max" value="35.55"/> -->
-    <xacro:property name="calf_torque_max" value="23.7"/>
+    <xacro:property name="calf_torque_max" value="35.55"/>
+    <!-- <xacro:property name="calf_torque_max" value="23.7"/> -->
     <xacro:property name="ros_version" value="$(env ROS_VERSION)" />
     <xacro:if value="${int(ros_version) == 1}">
